Commit message: fix(gazebo): split stereo sensors and bridge camera info

File: ros_ws/src/robots/descriptions/go2_description/xacro/realsense_d435i.xacro (robot description, xacro)
@@ -59,5 +59,11 @@
         <child link="camera_left_ir_frame"/>
     </joint>
-    <link name="camera_left_ir_frame"/>
+    <link name="camera_left_ir_frame">
+        <inertial>
+            <mass value="0.001"/>
+            <origin xyz="0 0 0" rpy="0 0 0"/>
+            <inertia ixx="1e-6" ixy="0" ixz="0" iyy="1e-6" iyz="0" izz="1e-6"/>
+        </inertial>
+    </link>
     <joint name="camera_left_ir_optical_joint" type="fixed">
         <origin xyz="0 0 0" rpy="-1.57079632679 0 -1.57079632679"/>
@@ -71,5 +77,11 @@
         <child link="camera_right_ir_frame"/>
     </joint>
-    <link name="camera_right_ir_frame"/>
+    <link name="camera_right_ir_frame">
+        <inertial>
+            <mass value="0.001"/>
+            <origin xyz="0 0 0" rpy="0 0 0"/>
+            <inertia ixx="1e-6" ixy="0" ixz="0" iyy="1e-6" iyz="0" izz="1e-6"/>
+        </inertial>
+    </link>
     <joint name="camera_right_ir_optical_joint" type="fixed">
         <origin xyz="0 0 0" rpy="-1.57079632679 0 -1.57079632679"/>
@@ -83,10 +95,18 @@
         <child link="camera_imu_frame"/>
     </joint>
-    <link name="camera_imu_frame"/>
-    <gazebo reference="camera_link">
+    <link name="camera_imu_frame">
+        <inertial>
+            <mass value="0.001"/>
+            <origin xyz="0 0 0" rpy="0 0 0"/>
+            <inertia ixx="1e-6" ixy="0" ixz="0" iyy="1e-6" iyz="0" izz="1e-6"/>
+        </inertial>
+    </link>
+    <gazebo reference="camera_color_frame">
         <sensor name="camera_color" type="camera">
+            <pose>0 0 0 0 0 0</pose>
             <always_on>true</always_on>
             <update_rate>30</update_rate>
             <topic>camera/color/image_raw</topic>
+            <camera_info_topic>camera/color/camera_info</camera_info_topic>
             <ignition_frame_id>camera_color_optical_frame</ignition_frame_id>
             <camera>
@@ -103,8 +123,12 @@
             </camera>
         </sensor>
+    </gazebo>
+    <gazebo reference="camera_depth_frame">
         <sensor name="camera_depth" type="depth_camera">
+            <pose>0 0 0 0 0 0</pose>
             <always_on>true</always_on>
             <update_rate>30</update_rate>
             <topic>camera/depth/image_raw</topic>
+            <camera_info_topic>camera/depth/camera_info</camera_info_topic>
             <ignition_frame_id>camera_depth_optical_frame</ignition_frame_id>
             <camera>
@@ -121,8 +145,12 @@
             </camera>
         </sensor>
+    </gazebo>
+    <gazebo reference="camera_left_ir_frame">
         <sensor name="camera_left_ir" type="camera">
+            <pose>0 0 0 0 0 0</pose>
             <always_on>true</always_on>
             <update_rate>30</update_rate>
             <topic>camera/infra1/image_raw</topic>
+            <camera_info_topic>camera/infra1/camera_info</camera_info_topic>
             <ignition_frame_id>camera_left_ir_optical_frame</ignition_frame_id>
             <camera>
@@ -139,8 +167,12 @@
             </camera>
         </sensor>
+    </gazebo>
+    <gazebo reference="camera_right_ir_frame">
         <sensor name="camera_right_ir" type="camera">
+            <pose>0 0 0 0 0 0</pose>
             <always_on>true</always_on>
             <update_rate>30</update_rate>
             <topic>camera/infra2/image_raw</topic>
+            <camera_info_topic>camera/infra2/camera_info</camera_info_topic>
             <ignition_frame_id>camera_right_ir_optical_frame</ignition_frame_id>
             <camera>
@@ -160,4 +192,5 @@
     <gazebo reference="camera_imu_frame">
         <sensor name="camera_imu_sensor" type="imu">
+            <pose>0 0 0 0 0 0</pose>
             <always_on>true</always_on>
             <update_rate>200</update_rate>

Commit message: feat(gazebo): visualize stereo rig and document 5cm baseline

File: ros_ws/src/robots/descriptions/go2_description/xacro/realsense_d435i.xacro (robot description, xacro)
@@ -5,5 +5,5 @@
          - horizontal FOV: 90 deg
          - intrinsics: fx = fy = 424, cx = 424, cy = 240
-         - current stereo baseline: 0.05 m -->
+         - stereo baseline: 0.05 m (left/right offsets are +/-0.025 m in Y) -->
     <joint name="camera_mount_joint" type="fixed">
         <origin xyz="0.245 0.0 0.045" rpy="0 0 0"/>
@@ -17,9 +17,13 @@
             <inertia ixx="1e-4" ixy="0" ixz="0" iyy="1e-4" iyz="0" izz="1e-4"/>
         </inertial>
-        <visual>
+        <visual name="camera_body_visual">
             <origin xyz="0 0 0" rpy="0 0 0"/>
             <geometry>
                 <box size="0.09 0.025 0.03"/>
             </geometry>
+            <material>
+                <ambient>0.2 0.2 0.2 1</ambient>
+                <diffuse>0.25 0.25 0.25 1</diffuse>
+            </material>
         </visual>
         <collision>
@@ -35,5 +39,16 @@
         <child link="camera_depth_frame"/>
     </joint>
-    <link name="camera_depth_frame"/>
+    <link name="camera_depth_frame">
+        <visual name="camera_depth_frustum_visual">
+            <origin xyz="0.06 0 0" rpy="0 0 0"/>
+            <geometry>
+                <mesh filename="file://$(find go2_description)/meshes/camera_frustum.dae" scale="0.12 0.12 0.12"/>
+            </geometry>
+            <material>
+                <ambient>0.1 0.6 1.0 0.35</ambient>
+                <diffuse>0.1 0.6 1.0 0.35</diffuse>
+            </material>
+        </visual>
+    </link>
     <joint name="camera_depth_optical_joint" type="fixed">
         <origin xyz="0 0 0" rpy="-1.57079632679 0 -1.57079632679"/>
@@ -65,4 +80,14 @@
             <inertia ixx="1e-6" ixy="0" ixz="0" iyy="1e-6" iyz="0" izz="1e-6"/>
         </inertial>
+        <visual name="camera_left_marker_visual">
+            <origin xyz="0 0 0" rpy="0 0 0"/>
+            <geometry>
+                <sphere radius="0.006"/>
+            </geometry>
+            <material>
+                <ambient>0.1 0.9 0.1 1</ambient>
+                <diffuse>0.1 0.9 0.1 1</diffuse>
+            </material>
+        </visual>
     </link>
     <joint name="camera_left_ir_optical_joint" type="fixed">
@@ -83,4 +108,14 @@
             <inertia ixx="1e-6" ixy="0" ixz="0" iyy="1e-6" iyz="0" izz="1e-6"/>
         </inertial>
+        <visual name="camera_right_marker_visual">
+            <origin xyz="0 0 0" rpy="0 0 0"/>
+            <geometry>
+                <sphere radius="0.006"/>
+            </geometry>
+            <material>
+                <ambient>0.9 0.1 0.1 1</ambient>
+                <diffuse>0.9 0.1 0.1 1</diffuse>
+            </material>
+        </visual>
     </link>
     <joint name="camera_right_ir_optical_joint" type="fixed">

Commit message: feat(gazebo): match tinynav realsense topic naming

File: ros_ws/src/robots/descriptions/go2_description/xacro/realsense_d435i.xacro (robot description, xacro)
@@ -41,12 +41,52 @@
     </joint>
     <link name="camera_depth_frame">
-        <visual name="camera_depth_frustum_visual">
-            <origin xyz="0.06 0 0" rpy="0 0 0"/>
-            <geometry>
-                <mesh filename="file://$(find go2_description)/meshes/camera_frustum.dae" scale="0.12 0.12 0.12"/>
-            </geometry>
-            <material>
-                <ambient>0.1 0.6 1.0 0.35</ambient>
-                <diffuse>0.1 0.6 1.0 0.35</diffuse>
+        <visual name="camera_depth_axis_visual">
+            <origin xyz="0.06 0 0" rpy="0 1.57079632679 0"/>
+            <geometry>
+                <cylinder radius="0.003" length="0.12"/>
+            </geometry>
+            <material>
+                <ambient>0.1 0.6 1.0 1</ambient>
+                <diffuse>0.1 0.6 1.0 1</diffuse>
+            </material>
+        </visual>
+        <visual name="camera_depth_fov_top_visual">
+            <origin xyz="0.06 0 0.06" rpy="0 0.78539816339 0"/>
+            <geometry>
+                <cylinder radius="0.0015" length="0.17"/>
+            </geometry>
+            <material>
+                <ambient>0.1 0.6 1.0 0.8</ambient>
+                <diffuse>0.1 0.6 1.0 0.8</diffuse>
+            </material>
+        </visual>
+        <visual name="camera_depth_fov_bottom_visual">
+            <origin xyz="0.06 0 -0.06" rpy="0 -0.78539816339 0"/>
+            <geometry>
+                <cylinder radius="0.0015" length="0.17"/>
+            </geometry>
+            <material>
+                <ambient>0.1 0.6 1.0 0.8</ambient>
+                <diffuse>0.1 0.6 1.0 0.8</diffuse>
+            </material>
+        </visual>
+        <visual name="camera_depth_fov_left_visual">
+            <origin xyz="0.06 0.06 0" rpy="1.57079632679 0.78539816339 0"/>
+            <geometry>
+                <cylinder radius="0.0015" length="0.17"/>
+            </geometry>
+            <material>
+                <ambient>0.1 0.6 1.0 0.8</ambient>
+                <diffuse>0.1 0.6 1.0 0.8</diffuse>
+            </material>
+        </visual>
+        <visual name="camera_depth_fov_right_visual">
+            <origin xyz="0.06 -0.06 0" rpy="1.57079632679 -0.78539816339 0"/>
+            <geometry>
+                <cylinder radius="0.0015" length="0.17"/>
+            </geometry>
+            <material>
+                <ambient>0.1 0.6 1.0 0.8</ambient>
+                <diffuse>0.1 0.6 1.0 0.8</diffuse>
             </material>
         </visual>
@@ -91,4 +131,14 @@
             </material>
         </visual>
+        <visual name="camera_left_axis_visual">
+            <origin xyz="0.04 0 0" rpy="0 1.57079632679 0"/>
+            <geometry>
+                <cylinder radius="0.002" length="0.08"/>
+            </geometry>
+            <material>
+                <ambient>0.1 0.9 0.1 1</ambient>
+                <diffuse>0.1 0.9 0.1 1</diffuse>
+            </material>
+        </visual>
     </link>
     <joint name="camera_left_ir_optical_joint" type="fixed">
@@ -113,4 +163,14 @@
             <geometry>
                 <sphere radius="0.006"/>
+            </geometry>
+            <material>
+                <ambient>0.9 0.1 0.1 1</ambient>
+                <diffuse>0.9 0.1 0.1 1</diffuse>
+            </material>
+        </visual>
+        <visual name="camera_right_axis_visual">
+            <origin xyz="0.04 0 0" rpy="0 1.57079632679 0"/>
+            <geometry>
+                <cylinder radius="0.002" length="0.08"/>
             </geometry>
             <material>

Commit message: fix(gazebo): make camera debug visuals larger and external

File: ros_ws/src/robots/descriptions/go2_description/xacro/realsense_d435i.xacro (robot description, xacro)
@@ -19,11 +19,11 @@
         </inertial>
         <visual name="camera_body_visual">
-            <origin xyz="0 0 0" rpy="0 0 0"/>
-            <geometry>
-                <box size="0.09 0.025 0.03"/>
-            </geometry>
-            <material>
-                <ambient>0.2 0.2 0.2 1</ambient>
-                <diffuse>0.25 0.25 0.25 1</diffuse>
+            <origin xyz="0.03 0 0" rpy="0 0 0"/>
+            <geometry>
+                <box size="0.12 0.03 0.04"/>
+            </geometry>
+            <material>
+                <ambient>0.95 0.65 0.1 1</ambient>
+                <diffuse>0.95 0.65 0.1 1</diffuse>
             </material>
         </visual>
@@ -42,7 +42,7 @@
     <link name="camera_depth_frame">
         <visual name="camera_depth_axis_visual">
-            <origin xyz="0.06 0 0" rpy="0 1.57079632679 0"/>
-            <geometry>
-                <cylinder radius="0.003" length="0.12"/>
+            <origin xyz="0.10 0 0" rpy="0 1.57079632679 0"/>
+            <geometry>
+                <cylinder radius="0.005" length="0.20"/>
             </geometry>
             <material>
@@ -52,41 +52,41 @@
         </visual>
         <visual name="camera_depth_fov_top_visual">
-            <origin xyz="0.06 0 0.06" rpy="0 0.78539816339 0"/>
-            <geometry>
-                <cylinder radius="0.0015" length="0.17"/>
-            </geometry>
-            <material>
-                <ambient>0.1 0.6 1.0 0.8</ambient>
-                <diffuse>0.1 0.6 1.0 0.8</diffuse>
+            <origin xyz="0.10 0 0.10" rpy="0 0.78539816339 0"/>
+            <geometry>
+                <cylinder radius="0.003" length="0.28"/>
+            </geometry>
+            <material>
+                <ambient>0.1 0.6 1.0 1</ambient>
+                <diffuse>0.1 0.6 1.0 1</diffuse>
             </material>
         </visual>
         <visual name="camera_depth_fov_bottom_visual">
-            <origin xyz="0.06 0 -0.06" rpy="0 -0.78539816339 0"/>
-            <geometry>
-                <cylinder radius="0.0015" length="0.17"/>
-            </geometry>
-            <material>
-                <ambient>0.1 0.6 1.0 0.8</ambient>
-                <diffuse>0.1 0.6 1.0 0.8</diffuse>
+            <origin xyz="0.10 0 -0.10" rpy="0 -0.78539816339 0"/>
+            <geometry>
+                <cylinder radius="0.003" length="0.28"/>
+            </geometry>
+            <material>
+                <ambient>0.1 0.6 1.0 1</ambient>
+                <diffuse>0.1 0.6 1.0 1</diffuse>
             </material>
         </visual>
         <visual name="camera_depth_fov_left_visual">
-            <origin xyz="0.06 0.06 0" rpy="1.57079632679 0.78539816339 0"/>
-            <geometry>
-                <cylinder radius="0.0015" length="0.17"/>
-            </geometry>
-            <material>
-                <ambient>0.1 0.6 1.0 0.8</ambient>
-                <diffuse>0.1 0.6 1.0 0.8</diffuse>
+            <origin xyz="0.10 0.10 0" rpy="1.57079632679 0.78539816339 0"/>
+            <geometry>
+                <cylinder radius="0.003" length="0.28"/>
+            </geometry>
+            <material>
+                <ambient>0.1 0.6 1.0 1</ambient>
+                <diffuse>0.1 0.6 1.0 1</diffuse>
             </material>
         </visual>
         <visual name="camera_depth_fov_right_visual">
-            <origin xyz="0.06 -0.06 0" rpy="1.57079632679 -0.78539816339 0"/>
-            <geometry>
-                <cylinder radius="0.0015" length="0.17"/>
-            </geometry>
-            <material>
-                <ambient>0.1 0.6 1.0 0.8</ambient>
-                <diffuse>0.1 0.6 1.0 0.8</diffuse>
+            <origin xyz="0.10 -0.10 0" rpy="1.57079632679 -0.78539816339 0"/>
+            <geometry>
+                <cylinder radius="0.003" length="0.28"/>
+            </geometry>
+            <material>
+                <ambient>0.1 0.6 1.0 1</ambient>
+                <diffuse>0.1 0.6 1.0 1</diffuse>
             </material>
         </visual>
@@ -122,21 +122,21 @@
         </inertial>
         <visual name="camera_left_marker_visual">
-            <origin xyz="0 0 0" rpy="0 0 0"/>
-            <geometry>
-                <sphere radius="0.006"/>
-            </geometry>
-            <material>
-                <ambient>0.1 0.9 0.1 1</ambient>
-                <diffuse>0.1 0.9 0.1 1</diffuse>
+            <origin xyz="0.05 0 0" rpy="0 0 0"/>
+            <geometry>
+                <sphere radius="0.012"/>
+            </geometry>
+            <material>
+                <ambient>0.1 0.95 0.1 1</ambient>
+                <diffuse>0.1 0.95 0.1 1</diffuse>
             </material>
         </visual>
         <visual name="camera_left_axis_visual">
-            <origin xyz="0.04 0 0" rpy="0 1.57079632679 0"/>
-            <geometry>
-                <cylinder radius="0.002" length="0.08"/>
-            </geometry>
-            <material>
-                <ambient>0.1 0.9 0.1 1</ambient>
-                <diffuse>0.1 0.9 0.1 1</diffuse>
+            <origin xyz="0.09 0 0" rpy="0 1.57079632679 0"/>
+            <geometry>
+                <cylinder radius="0.0035" length="0.10"/>
+            </geometry>
+            <material>
+                <ambient>0.1 0.95 0.1 1</ambient>
+                <diffuse>0.1 0.95 0.1 1</diffuse>
             </material>
         </visual>
@@ -160,21 +160,21 @@
         </inertial>
         <visual name="camera_right_marker_visual">
-            <origin xyz="0 0 0" rpy="0 0 0"/>
-            <geometry>
-                <sphere radius="0.006"/>
-            </geometry>
-            <material>
-                <ambient>0.9 0.1 0.1 1</ambient>
-                <diffuse>0.9 0.1 0.1 1</diffuse>
+            <origin xyz="0.05 0 0" rpy="0 0 0"/>
+            <geometry>
+                <sphere radius="0.012"/>
+            </geometry>
+            <material>
+                <ambient>0.95 0.1 0.1 1</ambient>
+                <diffuse>0.95 0.1 0.1 1</diffuse>
             </material>
         </visual>
         <visual name="camera_right_axis_visual">
-            <origin xyz="0.04 0 0" rpy="0 1.57079632679 0"/>
-            <geometry>
-                <cylinder radius="0.002" length="0.08"/>
-            </geometry>
-            <material>
-                <ambient>0.9 0.1 0.1 1</ambient>
-                <diffuse>0.9 0.1 0.1 1</diffuse>
+            <origin xyz="0.09 0 0" rpy="0 1.57079632679 0"/>
+            <geometry>
+                <cylinder radius="0.0035" length="0.10"/>
+            </geometry>
+            <material>
+                <ambient>0.95 0.1 0.1 1</ambient>
+                <diffuse>0.95 0.1 0.1 1</diffuse>
             </material>
         </visual>
