Commit message: fix(gazebo): add 1m xyz axes at stereo camera centers

File: ros_ws/src/robots/descriptions/go2_description/xacro/realsense_d435i.xacro (robot description, xacro)
@@ -40,56 +40,5 @@
         <child link="camera_depth_frame"/>
     </joint>
-    <link name="camera_depth_frame">
-        <visual name="camera_depth_axis_visual">
-            <origin xyz="0.10 0 0" rpy="0 1.57079632679 0"/>
-            <geometry>
-                <cylinder radius="0.005" length="0.20"/>
-            </geometry>
-            <material>
-                <ambient>0.1 0.6 1.0 1</ambient>
-                <diffuse>0.1 0.6 1.0 1</diffuse>
-            </material>
-        </visual>
-        <visual name="camera_depth_fov_top_visual">
-            <origin xyz="0.10 0 0.10" rpy="0 0.78539816339 0"/>
-            <geometry>
-                <cylinder radius="0.003" length="0.28"/>
-            </geometry>
-            <material>
-                <ambient>0.1 0.6 1.0 1</ambient>
-                <diffuse>0.1 0.6 1.0 1</diffuse>
-            </material>
-        </visual>
-        <visual name="camera_depth_fov_bottom_visual">
-            <origin xyz="0.10 0 -0.10" rpy="0 -0.78539816339 0"/>
-            <geometry>
-                <cylinder radius="0.003" length="0.28"/>
-            </geometry>
-            <material>
-                <ambient>0.1 0.6 1.0 1</ambient>
-                <diffuse>0.1 0.6 1.0 1</diffuse>
-            </material>
-        </visual>
-        <visual name="camera_depth_fov_left_visual">
-            <origin xyz="0.10 0.10 0" rpy="1.57079632679 0.78539816339 0"/>
-            <geometry>
-                <cylinder radius="0.003" length="0.28"/>
-            </geometry>
-            <material>
-                <ambient>0.1 0.6 1.0 1</ambient>
-                <diffuse>0.1 0.6 1.0 1</diffuse>
-            </material>
-        </visual>
-        <visual name="camera_depth_fov_right_visual">
-            <origin xyz="0.10 -0.10 0" rpy="1.57079632679 -0.78539816339 0"/>
-            <geometry>
-                <cylinder radius="0.003" length="0.28"/>
-            </geometry>
-            <material>
-                <ambient>0.1 0.6 1.0 1</ambient>
-                <diffuse>0.1 0.6 1.0 1</diffuse>
-            </material>
-        </visual>
-    </link>
+    <link name="camera_depth_frame"/>
     <joint name="camera_depth_optical_joint" type="fixed">
         <origin xyz="0 0 0" rpy="-1.57079632679 0 -1.57079632679"/>
@@ -121,22 +70,32 @@
             <inertia ixx="1e-6" ixy="0" ixz="0" iyy="1e-6" iyz="0" izz="1e-6"/>
         </inertial>
-        <visual name="camera_left_marker_visual">
-            <origin xyz="0.05 0 0" rpy="0 0 0"/>
-            <geometry>
-                <sphere radius="0.012"/>
-            </geometry>
-            <material>
-                <ambient>0.1 0.95 0.1 1</ambient>
-                <diffuse>0.1 0.95 0.1 1</diffuse>
-            </material>
-        </visual>
-        <visual name="camera_left_axis_visual">
-            <origin xyz="0.09 0 0" rpy="0 1.57079632679 0"/>
-            <geometry>
-                <cylinder radius="0.0035" length="0.10"/>
-            </geometry>
-            <material>
-                <ambient>0.1 0.95 0.1 1</ambient>
-                <diffuse>0.1 0.95 0.1 1</diffuse>
+        <visual name="camera_left_x_axis_visual">
+            <origin xyz="0.5 0 0" rpy="0 1.57079632679 0"/>
+            <geometry>
+                <cylinder radius="0.008" length="1.0"/>
+            </geometry>
+            <material>
+                <ambient>1 0 0 1</ambient>
+                <diffuse>1 0 0 1</diffuse>
+            </material>
+        </visual>
+        <visual name="camera_left_y_axis_visual">
+            <origin xyz="0 0.5 0" rpy="1.57079632679 0 0"/>
+            <geometry>
+                <cylinder radius="0.008" length="1.0"/>
+            </geometry>
+            <material>
+                <ambient>0 1 0 1</ambient>
+                <diffuse>0 1 0 1</diffuse>
+            </material>
+        </visual>
+        <visual name="camera_left_z_axis_visual">
+            <origin xyz="0 0 0.5" rpy="0 0 0"/>
+            <geometry>
+                <cylinder radius="0.008" length="1.0"/>
+            </geometry>
+            <material>
+                <ambient>0 0 1 1</ambient>
+                <diffuse>0 0 1 1</diffuse>
             </material>
         </visual>
@@ -159,22 +118,32 @@
             <inertia ixx="1e-6" ixy="0" ixz="0" iyy="1e-6" iyz="0" izz="1e-6"/>
         </inertial>
-        <visual name="camera_right_marker_visual">
-            <origin xyz="0.05 0 0" rpy="0 0 0"/>
-            <geometry>
-                <sphere radius="0.012"/>
-            </geometry>
-            <material>
-                <ambient>0.95 0.1 0.1 1</ambient>
-                <diffuse>0.95 0.1 0.1 1</diffuse>
-            </material>
-        </visual>
-        <visual name="camera_right_axis_visual">
-            <origin xyz="0.09 0 0" rpy="0 1.57079632679 0"/>
-            <geometry>
-                <cylinder radius="0.0035" length="0.10"/>
-            </geometry>
-            <material>
-                <ambient>0.95 0.1 0.1 1</ambient>
-                <diffuse>0.95 0.1 0.1 1</diffuse>
+        <visual name="camera_right_x_axis_visual">
+            <origin xyz="0.5 0 0" rpy="0 1.57079632679 0"/>
+            <geometry>
+                <cylinder radius="0.008" length="1.0"/>
+            </geometry>
+            <material>
+                <ambient>1 0 0 1</ambient>
+                <diffuse>1 0 0 1</diffuse>
+            </material>
+        </visual>
+        <visual name="camera_right_y_axis_visual">
+            <origin xyz="0 0.5 0" rpy="1.57079632679 0 0"/>
+            <geometry>
+                <cylinder radius="0.008" length="1.0"/>
+            </geometry>
+            <material>
+                <ambient>0 1 0 1</ambient>
+                <diffuse>0 1 0 1</diffuse>
+            </material>
+        </visual>
+        <visual name="camera_right_z_axis_visual">
+            <origin xyz="0 0 0.5" rpy="0 0 0"/>
+            <geometry>
+                <cylinder radius="0.008" length="1.0"/>
+            </geometry>
+            <material>
+                <ambient>0 0 1 1</ambient>
+                <diffuse>0 0 1 1</diffuse>
             </material>
         </visual>

Commit message: revert(gazebo): drop non-working camera debug visuals

File: ros_ws/src/robots/descriptions/go2_description/xacro/realsense_d435i.xacro (robot description, xacro)
@@ -19,11 +19,11 @@
         </inertial>
         <visual name="camera_body_visual">
-            <origin xyz="0.03 0 0" rpy="0 0 0"/>
-            <geometry>
-                <box size="0.12 0.03 0.04"/>
-            </geometry>
-            <material>
-                <ambient>0.95 0.65 0.1 1</ambient>
-                <diffuse>0.95 0.65 0.1 1</diffuse>
+            <origin xyz="0 0 0" rpy="0 0 0"/>
+            <geometry>
+                <box size="0.09 0.025 0.03"/>
+            </geometry>
+            <material>
+                <ambient>0.2 0.2 0.2 1</ambient>
+                <diffuse>0.25 0.25 0.25 1</diffuse>
             </material>
         </visual>
@@ -40,5 +40,56 @@
         <child link="camera_depth_frame"/>
     </joint>
-    <link name="camera_depth_frame"/>
+    <link name="camera_depth_frame">
+        <visual name="camera_depth_axis_visual">
+            <origin xyz="0.06 0 0" rpy="0 1.57079632679 0"/>
+            <geometry>
+                <cylinder radius="0.003" length="0.12"/>
+            </geometry>
+            <material>
+                <ambient>0.1 0.6 1.0 1</ambient>
+                <diffuse>0.1 0.6 1.0 1</diffuse>
+            </material>
+        </visual>
+        <visual name="camera_depth_fov_top_visual">
+            <origin xyz="0.06 0 0.06" rpy="0 0.78539816339 0"/>
+            <geometry>
+                <cylinder radius="0.0015" length="0.17"/>
+            </geometry>
+            <material>
+                <ambient>0.1 0.6 1.0 0.8</ambient>
+                <diffuse>0.1 0.6 1.0 0.8</diffuse>
+            </material>
+        </visual>
+        <visual name="camera_depth_fov_bottom_visual">
+            <origin xyz="0.06 0 -0.06" rpy="0 -0.78539816339 0"/>
+            <geometry>
+                <cylinder radius="0.0015" length="0.17"/>
+            </geometry>
+            <material>
+                <ambient>0.1 0.6 1.0 0.8</ambient>
+                <diffuse>0.1 0.6 1.0 0.8</diffuse>
+            </material>
+        </visual>
+        <visual name="camera_depth_fov_left_visual">
+            <origin xyz="0.06 0.06 0" rpy="1.57079632679 0.78539816339 0"/>
+            <geometry>
+                <cylinder radius="0.0015" length="0.17"/>
+            </geometry>
+            <material>
+                <ambient>0.1 0.6 1.0 0.8</ambient>
+                <diffuse>0.1 0.6 1.0 0.8</diffuse>
+            </material>
+        </visual>
+        <visual name="camera_depth_fov_right_visual">
+            <origin xyz="0.06 -0.06 0" rpy="1.57079632679 -0.78539816339 0"/>
+            <geometry>
+                <cylinder radius="0.0015" length="0.17"/>
+            </geometry>
+            <material>
+                <ambient>0.1 0.6 1.0 0.8</ambient>
+                <diffuse>0.1 0.6 1.0 0.8</diffuse>
+            </material>
+        </visual>
+    </link>
     <joint name="camera_depth_optical_joint" type="fixed">
         <origin xyz="0 0 0" rpy="-1.57079632679 0 -1.57079632679"/>
@@ -70,32 +121,22 @@
             <inertia ixx="1e-6" ixy="0" ixz="0" iyy="1e-6" iyz="0" izz="1e-6"/>
         </inertial>
-        <visual name="camera_left_x_axis_visual">
-            <origin xyz="0.5 0 0" rpy="0 1.57079632679 0"/>
-            <geometry>
-                <cylinder radius="0.008" length="1.0"/>
-            </geometry>
-            <material>
-                <ambient>1 0 0 1</ambient>
-                <diffuse>1 0 0 1</diffuse>
-            </material>
-        </visual>
-        <visual name="camera_left_y_axis_visual">
-            <origin xyz="0 0.5 0" rpy="1.57079632679 0 0"/>
-            <geometry>
-                <cylinder radius="0.008" length="1.0"/>
-            </geometry>
-            <material>
-                <ambient>0 1 0 1</ambient>
-                <diffuse>0 1 0 1</diffuse>
-            </material>
-        </visual>
-        <visual name="camera_left_z_axis_visual">
-            <origin xyz="0 0 0.5" rpy="0 0 0"/>
-            <geometry>
-                <cylinder radius="0.008" length="1.0"/>
-            </geometry>
-            <material>
-                <ambient>0 0 1 1</ambient>
-                <diffuse>0 0 1 1</diffuse>
+        <visual name="camera_left_marker_visual">
+            <origin xyz="0 0 0" rpy="0 0 0"/>
+            <geometry>
+                <sphere radius="0.006"/>
+            </geometry>
+            <material>
+                <ambient>0.1 0.9 0.1 1</ambient>
+                <diffuse>0.1 0.9 0.1 1</diffuse>
+            </material>
+        </visual>
+        <visual name="camera_left_axis_visual">
+            <origin xyz="0.04 0 0" rpy="0 1.57079632679 0"/>
+            <geometry>
+                <cylinder radius="0.002" length="0.08"/>
+            </geometry>
+            <material>
+                <ambient>0.1 0.9 0.1 1</ambient>
+                <diffuse>0.1 0.9 0.1 1</diffuse>
             </material>
         </visual>
@@ -118,32 +159,22 @@
             <inertia ixx="1e-6" ixy="0" ixz="0" iyy="1e-6" iyz="0" izz="1e-6"/>
         </inertial>
-        <visual name="camera_right_x_axis_visual">
-            <origin xyz="0.5 0 0" rpy="0 1.57079632679 0"/>
-            <geometry>
-                <cylinder radius="0.008" length="1.0"/>
-            </geometry>
-            <material>
-                <ambient>1 0 0 1</ambient>
-                <diffuse>1 0 0 1</diffuse>
-            </material>
-        </visual>
-        <visual name="camera_right_y_axis_visual">
-            <origin xyz="0 0.5 0" rpy="1.57079632679 0 0"/>
-            <geometry>
-                <cylinder radius="0.008" length="1.0"/>
-            </geometry>
-            <material>
-                <ambient>0 1 0 1</ambient>
-                <diffuse>0 1 0 1</diffuse>
-            </material>
-        </visual>
-        <visual name="camera_right_z_axis_visual">
-            <origin xyz="0 0 0.5" rpy="0 0 0"/>
-            <geometry>
-                <cylinder radius="0.008" length="1.0"/>
-            </geometry>
-            <material>
-                <ambient>0 0 1 1</ambient>
-                <diffuse>0 0 1 1</diffuse>
+        <visual name="camera_right_marker_visual">
+            <origin xyz="0 0 0" rpy="0 0 0"/>
+            <geometry>
+                <sphere radius="0.006"/>
+            </geometry>
+            <material>
+                <ambient>0.9 0.1 0.1 1</ambient>
+                <diffuse>0.9 0.1 0.1 1</diffuse>
+            </material>
+        </visual>
+        <visual name="camera_right_axis_visual">
+            <origin xyz="0.04 0 0" rpy="0 1.57079632679 0"/>
+            <geometry>
+                <cylinder radius="0.002" length="0.08"/>
+            </geometry>
+            <material>
+                <ambient>0.9 0.1 0.1 1</ambient>
+                <diffuse>0.9 0.1 0.1 1</diffuse>
             </material>
         </visual>

Commit message: fix(gazebo): align camera imu frame with left infrared frame

File: ros_ws/src/robots/descriptions/go2_description/xacro/realsense_d435i.xacro (robot description, xacro)
@@ -188,5 +188,5 @@
     <joint name="camera_imu_joint" type="fixed">
         <origin xyz="0 0 0" rpy="0 0 0"/>
-        <parent link="camera_link"/>
+        <parent link="camera_left_ir_frame"/>
         <child link="camera_imu_frame"/>
     </joint>

Commit message: fix(gazebo): align camera imu frame with left infrared optical frame

File: ros_ws/src/robots/descriptions/go2_description/xacro/realsense_d435i.xacro (robot description, xacro)
@@ -188,5 +188,5 @@
     <joint name="camera_imu_joint" type="fixed">
         <origin xyz="0 0 0" rpy="0 0 0"/>
-        <parent link="camera_left_ir_frame"/>
+        <parent link="camera_left_ir_optical_frame"/>
         <child link="camera_imu_frame"/>
     </joint>
